File: Hardware/IotaWatt4.8.brd (EAGLE design)
At the start: 80 x 113 mm, 58 parts, among them J0 2.1MMJACKSMT, J1 STEREO_SMD, J10 STEREO_SMD, J11 STEREO_SMD, J12 STEREO_SMD, J13 STEREO_SMD, J14 STEREO_SMD, J2 STEREO_SMD, J3 STEREO_SMD, J4 STEREO_SMD, J5 STEREO_SMD, J6 STEREO_SMD, J7 STEREO_SMD, J8 STEREO_SMD, J9 STEREO_SMD, Y1 32Khz

Commit message: Post my changes again
Parts:
- added U$5: ESP32DEVKITV1, ESP32-DEVKITV1:ESP32-DEVKITV1
- moved J0 2.40 mm to (57.4, 2.37)
- moved U$16 1.50 mm to (33.8, 24.4)
- moved C5 0.92 mm to (43.6, 49.9), turned to 0 degrees
- moved U$23 0.81 mm to (18.2, 4.65)
- moved R4 0.70 mm to (18.1, 9.00)
Connections:
- removed net N$10: R4.2, U$16.P$30
- new net LED: R4.2, U$16.P$30, U$5.15
- net 3V3: now also U$5.1
- net ADCCS0: now also U$5.11
- net ADCCS1: now also U$5.12
- net CSSD: now also U$5.3
- net GND: now also U$5.2, U$5.28
- net MISO: now also U$5.27
- net MOSI: now also U$5.28
- net SCL: now also U$5.14
- net SCLK: now also U$5.26
- net SDA: now also U$5.13
Routing:
- net LED: track 0.00 -> 65.3 mm, vias 0 -> 1
- net N$10: track 58.3 -> 0.00 mm, vias 1 -> 0
- net MOSI: track 112.3 -> 132.6 mm, vias 3 -> 5
- net SCLK: track 118.1 -> 138.2 mm, vias 2 -> 4
- net MISO: track 126.4 -> 144.4 mm, vias 3 -> 5
- net 3V3: track 323.1 -> 334.1 mm
- net SCL: track 41.1 -> 49.3 mm
- net SDA: track 42.3 -> 49.9 mm
- net ADCCS1: track 85.8 -> 91.6 mm
- net ADCCS0: track 35.9 -> 39.7 mm
- net CSSD: track 113.4 -> 116.3 mm
- net N$27: track 17.5 -> 16.3 mm
- net ACBIAS: track 91.5 -> 92.2 mm
- net GND: vias 59 -> 60
Other:
- board text added: "Rev 4.8b"
- board text added: "dotnetdan"
- board text removed: "Rev 4.8"
- board text removed: "genuine"
- board text removed: "tm"
