File: Hardware/IotaWatt4.8.sch (EAGLE design)
At the start: 58 parts, among them J0 2.1MMJACKSMT, J1 STEREO_SMD, J10 STEREO_SMD, J11 STEREO_SMD, J12 STEREO_SMD, J13 STEREO_SMD, J14 STEREO_SMD, J2 STEREO_SMD, J3 STEREO_SMD, J4 STEREO_SMD, J5 STEREO_SMD, J6 STEREO_SMD, J7 STEREO_SMD, J8 STEREO_SMD, J9 STEREO_SMD, Y1 32Khz

Commit message: Post my changes again
Parts:
- added U$5: ESP32DEVKITV1, ESP32-DEVKITV1:ESP32DEVKITV1
Connections:
- removed net N$10: R4.2, U$16.GPIO16
- new net LED: R4.2, U$16.GPIO16, U$5.IO23
- net 3V3: now also U$5.3V3
- net ADCCS0: now also U$5.IO21
- net ADCCS1: now also U$5.IO3
- net CSSD: now also U$5.IO15
- net GND: now also U$5.GND, U$5.GND1
- net MISO: now also U$5.IO12
- net MOSI: now also U$5.IO13
- net SCL: now also U$5.IO22
- net SCLK: now also U$5.IO14
- net SDA: now also U$5.IO1
Changed lines of the file:
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@@
 <?xml version="1.0" encoding="utf-8"?>
 <!DOCTYPE eagle SYSTEM "eagle.dtd">
-<eagle version="8.1.1">
+<eagle version="7.2.0">
 <drawing>
 <settings>
@@
 <layer number="59" name="tCarbon" color="7" fill="1" visible="no" active="no"/>
 <layer number="60" name="bCarbon" color="7" fill="1" visible="no" active="no"/>
+<layer number="88" name="SimResults" color="9" fill="1" visible="yes" active="yes"/>
+<layer number="89" name="SimProbes" color="9" fill="1" visible="yes" active="yes"/>
 <layer number="90" name="Modules" color="5" fill="1" visible="yes" active="yes"/>
 <layer number="91" name="Nets" color="2" fill="1" visible="yes" active="yes"/>
@@
 <part name="C7" library="adafruit" deviceset="C-US" device="C0805" value="10uF"/>
 <part name="R3" library="adafruit" deviceset="R-US_" device="R0805" value="1K"/>
+<part name="U$5" library="ESP32-DEVKITV1" deviceset="ESP32DEVKITV1" device=""/>
 </parts>
 <sheets>
@@
 <attribute name="VALUE" x="162.814" y="11.938" size="1.778" layer="96"/>
 </instance>
+<instance part="U$5" gate="G$1" x="241.3" y="93.98" rot="R90"/>
 </instances>
 <busses>
@@
 <wire x1="160.02" y1="25.4" x2="157.48" y2="25.4" width="0.1524" layer="91"/>
 </segment>
+<segment>
+<pinref part="U$5" gate="G$1" pin="GND"/>
+<wire x1="259.08" y1="73.66" x2="264.16" y2="73.66" width="0.1524" layer="91"/>
+</segment>
+<segment>
+<pinref part="U$5" gate="G$1" pin="GND1"/>
+<wire x1="223.52" y1="73.66" x2="218.44" y2="73.66" width="0.1524" layer="91"/>
+</segment>
 </net>
 <net name="ADC1" class="0">
@@
 <label x="213.36" y="30.48" size="1.778" layer="91" xref="yes"/>
 </segment>
+<segment>
+<pinref part="U$5" gate="G$1" pin="IO12"/>
+<wire x1="223.52" y1="78.74" x2="218.44" y2="78.74" width="0.1524" layer="91"/>
+</segment>
 </net>
 <net name="MOSI" class="0">
@@
 <label x="190.5" y="25.4" size="1.778" layer="91" rot="R180" xref="yes"/>
 </segment>
+<segment>
+<pinref part="U$5" gate="G$1" pin="IO13"/>
+<wire x1="223.52" y1="76.2" x2="218.44" y2="76.2" width="0.1524" layer="91"/>
+</segment>
 </net>
 <net name="SCLK" class="0">
@@
 <junction x="213.36" y="20.32"/>
 <label x="213.36" y="20.32" size="1.778" layer="91" xref="yes"/>
+</segment>
+<segment>
+<pinref part="U$5" gate="G$1" pin="IO14"/>
+<wire x1="223.52" y1="81.28" x2="218.44" y2="81.28" width="0.1524" layer="91"/>
 </segment>
 </net>
@@
 <junction x="170.18" y="15.24"/>
 </segment>
+<segment>
+<pinref part="U$5" gate="G$1" pin="3V3"/>
+<wire x1="259.08" y1="71.12" x2="264.16" y2="71.12" width="0.1524" layer="91"/>
+</segment>
 </net>
 <net name="ADC7" class="0">
@@
 <wire x1="185.42" y1="104.14" x2="185.42" y2="83.82" width="0.1524" layer="91"/>
 </segment>
+<segment>
+<pinref part="U$5" gate="G$1" pin="IO3"/>
+<wire x1="259.08" y1="99.06" x2="264.16" y2="99.06" width="0.1524" layer="91"/>
+</segment>
 </net>
 <net name="N$27" class="0">
@@
 <label x="157.48" y="83.82" size="1.778" layer="91" xref="yes"/>
 </segment>
+<segment>
+<pinref part="U$5" gate="G$1" pin="IO21"/>
+<wire x1="259.08" y1="96.52" x2="264.16" y2="96.52" width="0.1524" layer="91"/>
+</segment>
 </net>
 <net name="CSSD" class="0">
@@
 <junction x="190.5" y="30.48"/>
 <label x="190.5" y="30.48" size="1.778" layer="91" rot="R180" xref="yes"/>
+</segment>
+<segment>
+<pinref part="U$5" gate="G$1" pin="IO15"/>
+<wire x1="259.08" y1="76.2" x2="264.16" y2="76.2" width="0.1524" layer="91"/>
 </segment>
 </net>
@@
 <wire x1="157.48" y1="7.62" x2="157.48" y2="5.08" width="0.1524" layer="91"/>
 </segment>
+<segment>
+<pinref part="U$5" gate="G$1" pin="IO1"/>
+<wire x1="259.08" y1="101.6" x2="264.16" y2="101.6" width="0.1524" layer="91"/>
+</segment>
 </net>
 <net name="SCL" class="0">
@@
 <label x="157.48" y="10.16" size="1.778" layer="91" xref="yes"/>
 <wire x1="152.4" y1="10.16" x2="157.48" y2="10.16" width="0.1524" layer="91"/>
+</segment>
+<segment>
+<pinref part="U$5" gate="G$1" pin="IO22"/>
+<wire x1="259.08" y1="104.14" x2="264.16" y2="104.14" width="0.1524" layer="91"/>
 </segment>
 </net>
@@
 </segment>
 </net>
-<net name="N$10" class="0">
+<net name="LED" class="0">
 <segment>
 <pinref part="U$16" gate="G$1" pin="GPIO16"/>
@@
 <junction x="165.1" y="104.14"/>
 </segment>
-</net>
+<segment>
+<pinref part="U$5" gate="G$1" pin="IO23"/>
+<wire x1="259.08" y1="106.68" x2="264.16" y2="106.68" width="0.1524" layer="91"/>
+</segment>
+</net>
